Commit message: Readded the LIDAR
The LIDAR was added back in for using SLAM

File: scamp_ws/src/turtlebot3_description/urdf/turtlebot3_waffle_pi.gazebo.xacro (robot description, xacro)
@@ -102,5 +102,5 @@
     </plugin>
   </gazebo>
-  <!--<gazebo reference="base_scan">
+  <gazebo reference="base_scan">
     <material>Gazebo/FlatBlack</material>
     <sensor type="ray" name="lds_lfcd_sensor">
@@ -133,5 +133,5 @@
       </plugin>
     </sensor>
-  </gazebo>-->
+  </gazebo>
 <!--link : https://www.raspberrypi.org/documentation/hardware/camera/-->
   <gazebo reference="camera_rgb_frame">

File: scamp_ws/src/turtlebot3_description/urdf/turtlebot3_waffle_pi.urdf.xacro (robot description, xacro)
@@ -133,5 +133,5 @@
   </joint>
   <link name="imu_link"/>
-  <!--<joint name="scan_joint" type="fixed">
+  <joint name="scan_joint" type="fixed">
     <parent link="base_link"/>
     <child link="base_scan"/>
@@ -159,5 +159,5 @@
                izz="0.001" />
     </inertial>
-  </link>-->
+  </link>
   <joint name="camera_joint" type="fixed">
     <origin xyz="0.073 -0.011 0.084" rpy="0 0 0"/>
